File: robocup2027-pcb-data.kicad_sch (KiCad schematic)
At the start: 46 parts, among them M5 Motor_Servo, M6 Motor_Servo, Q1 BPW40, Q2 BPW40, U1 ESP32-DEVKITC-32E

Commit message: assigned footprints and added them to pcb
Parts:
- U13: footprint (none) -> robo:fe-urt-2
Changed lines of the file:
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@@
 			)
 		)
-		(property "Footprint" ""
+		(property "Footprint" "robo:fe-urt-2"
 			(at 314.96 35.56 0)
 			(effects

Commit message: update
Parts:
- S1, S2: footprint robo:DS-850K-S-ON -> robo:CW-SB11KKFF
Changed lines of the file:
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@@
 			)
 		)
-		(property "Footprint" "robo:DS-850K-S-ON"
+		(property "Footprint" "robo:CW-SB11KKFF"
 			(at 86.36 133.35 0)
 			(effects
@@
 			)
 		)
-		(property "Footprint" "robo:DS-850K-S-ON"
+		(property "Footprint" "robo:CW-SB11KKFF"
 			(at 38.1 38.1 0)
 			(effects

Commit message: placing bno550
Parts:
- added U14: ~, robo:AE-BNO055-BO, symbol robo:AE-BNO055-BO
Connections:
- net +3.3V: now also U14.1 (VIN)
- net GND: now also U14.2 (GND), U14.7 (GND)
- net I2C_SCL: now also U14.4 (SCL/R)
- net I2C_SDA: now also U14.3 (SDA/T)
- no-connect marks 49 -> 52

Commit message: update
Connections:
- net XSHUT2: now reaches U7.5 (XSHUT)
- net XSHUT2: now also U1.J3_9 (IO18)
- net XSHUT1: now reaches U1.J2_12 (IO14)
- net XSHUT1: now also U6.5 (XSHUT)
- net XSHUT5: now reaches U1.J3_10 (IO5)
- net XSHUT5: now also U10.5 (XSHUT)
- net XSHUT6: now reaches U1.J3_16 (IO15)
- net XSHUT6: now also U15.5 (XSHUT)
- net XSHUT4: now reaches U1.J3_2 (IO23)
- net XSHUT4: now also U9.5 (XSHUT)
- net XSHUT3: now reaches U1.J3_8 (IO19)
- net XSHUT3: now also U8.5 (XSHUT)
- no-connect marks 52 -> 40
Other:
- note added: "gyro"

Commit message: add debug speaker
Parts:
- added U17: ~, robo:PKM13EPYH4000-A0, symbol robo:PKM13EPYH4000-A0
- Q1, Q2: footprint robo:2.54mm_capacitor -> LED_THT:LED_D5.0mm_Clear
- S1, S2: footprint robo:CW-SB11KKFF -> 4-1437565-0:SW_4-1437565-0
- U1: footprint robo:MODULE_ESP32-DEVKITC-32E -> ESP32-DEVKITC-32E:MODULE_ESP32-DEVKITC-32E
Connections:
- net GND: now also U17.1 (GND)
- net Debug: now reaches U1.J3_15 (IO2)
- net Debug: now also U17.2 (VCC)
- no-connect marks 40 -> 39
Changed lines of the file:
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@@
 	)
 	(no_connect
-		(at 134.62 158.75)
-	)
-	(no_connect
 		(at 93.98 161.29)
 	)
@@
 		)
 	)
+	(global_label "Debug"
+		(shape output)
+		(at 134.62 158.75 0)
+		(fields_autoplaced yes)
+		(effects
+			(font
+				(size 1.27 1.27)
+			)
+			(justify left)
+		)
+		(property "Intersheetrefs" "${INTERSHEET_REFS}"
+			(at 143.4108 158.75 0)
+			(effects
+				(font
+					(size 1.27 1.27)
+				)
+				(justify left)
+				(hide yes)
+			)
+		)
+	)
 	(global_label "XSHUT5"
 		(shape input)
@@
 		)
 	)
+	(global_label "Debug"
+		(shape input)
+		(at 168.91 173.99 270)
+		(fields_autoplaced yes)
+		(effects
+			(font
+				(size 1.27 1.27)
+			)
+			(justify right)
+		)
+		(property "Intersheetrefs" "${INTERSHEET_REFS}"
+			(at 168.91 182.7808 90)
+			(effects
+				(font
+					(size 1.27 1.27)
+				)
+				(justify right)
+				(hide yes)
+			)
+		)
+	)
 	(global_label "FE-URT-2-RXD"
 		(shape input)
@@
 			)
 		)
-		(property "Footprint" "robo:MODULE_ESP32-DEVKITC-32E"
+		(property "Footprint" "ESP32-DEVKITC-32E:MODULE_ESP32-DEVKITC-32E"
 			(at 114.3 146.05 0)
 			(effects
@@
 			)
 		)
-		(property "Footprint" "robo:2.54mm_capacitor"
+		(property "Footprint" "LED_THT:LED_D5.0mm_Clear"
 			(at 247.904 47.752 0)
 			(effects
@@
 			)
 		)
-		(property "Footprint" "robo:2.54mm_capacitor"
+		(property "Footprint" "LED_THT:LED_D5.0mm_Clear"
 			(at 247.904 64.262 0)
 			(effects
@@
 			)
 		)
-		(property "Footprint" "robo:CW-SB11KKFF"
+		(property "Footprint" "4-1437565-0:SW_4-1437565-0"
 			(at 86.36 133.35 0)
 			(effects
@@
 	)
 	(symbol
-		(lib_name "DCDC-3.3v_1")
 		(lib_id "robo:DCDC-3.3v")
 		(at 101.6 36.83 270)
@@
 	)
 	(symbol
+		(lib_id "power:GND")
+		(at 166.37 173.99 0)
+		(unit 1)
+		(exclude_from_sim no)
+		(in_bom yes)
+		(on_board yes)
+		(dnp no)
+		(fields_autoplaced yes)
+		(property "Reference" "#PWR029"
+			(at 166.37 180.34 0)
+			(effects
+				(font
+					(size 1.27 1.27)
+				)
+				(hide yes)
+			)
+		)
+		(property "Value" "GND"
+			(at 166.37 179.07 0)
+			(effects
+				(font
+					(size 1.27 1.27)
+				)
+			)
+		)
+		(property "Footprint" ""
+			(at 166.37 173.99 0)
+			(effects
+				(font
+					(size 1.27 1.27)
+				)
+				(hide yes)
+			)
+		)
+		(property "Datasheet" ""
+			(at 166.37 173.99 0)
+			(effects
+				(font
+					(size 1.27 1.27)
+				)
+				(hide yes)
+			)
+		)
+		(property "Description" "Power symbol creates a global label with name \"GND\" , ground"
+			(at 166.37 173.99 0)
+			(effects
+				(font
+					(size 1.27 1.27)
+				)
+				(hide yes)
+			)
+		)
+		(pin "1"
+		)
+		(instances
+			(project "robocup2027-pcb-data"
+				(path "/fda8bdee-4e79-4e78-9174-7c0702f316a4"
+					(reference "#PWR029")
+					(unit 1)
+				)
+			)
+		)
+	)
+	(symbol
 		(lib_id "power:+6V")
 		(at 97.79 73.66 0)
@@
 			)
 		)
-		(property "Footprint" "robo:CW-SB11KKFF"
+		(property "Footprint" "4-1437565-0:SW_4-1437565-0"
 			(at 38.1 38.1 0)
 			(effects
@@
 					(unit 1)
 				)
+			)
+		)
+	)
+	(symbol
+		(lib_id "robo:PKM13EPYH4000-A0")
+		(at 167.64 171.45 0)
+		(unit 1)
+		(exclude_from_sim no)
+		(in_bom yes)
+		(on_board yes)
+		(dnp no)
+		(fields_autoplaced yes)
+		(property "Reference" "U17"
+			(at 170.18 169.5449 0)
+			(effects
+				(font
+					(size 1.27 1.27)
+				)
+				(justify left)
+			)
+		)
+		(property "Value" "~"
+			(at 170.18 172.0849 0)
+			(effects
+				(font
+					(size 1.27 1.27)
+				)
+				(justify left)
+			)
+		)
+		(property "Footprint" "robo:PKM13EPYH4000-A0"
+			(at 167.64 171.45 0)
+			(effects
+				(font
+					(size 1.27 1.27)
+				)
+				(hide yes)
+			)
+		)
+		(property "Datasheet" ""
+			(at 167.64 171.45 0)
+			(effects
+				(font
+					(size 1.27 1.27)
+				)
+				(hide yes)
+			)
+		)
+		(property "Description" ""
+			(at 167.64 171.45 0)
+			(effects
+				(font
+					(size 1.27 1.27)
+				)
+				(hide yes)
+			)
+		)
+		(pin "1"
+		)
+		(pin "2"
+		)
+		(instances
+			(project ""
+				(path "/fda8bdee-4e79-4e78-9174-7c0702f316a4"
+					(reference "U17")
+					(unit 1)
+				)

Commit message: finished tracing
Parts:
- S1, S2: footprint 4-1437565-0:SW_4-1437565-0 -> robo:CW-SB11KKFF
- U1: footprint ESP32-DEVKITC-32E:MODULE_ESP32-DEVKITC-32E -> robo:MODULE_ESP32-DEVKITC-32E
Connections:
- net +3.3V: now also U13.3 (5V)
- net +5V: no longer U13.3 (5V)
Changed lines of the file:
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@@
 	)
 	(symbol
-		(lib_id "power:+5V")
-		(at 303.53 25.4 0)
-		(unit 1)
-		(exclude_from_sim no)
-		(in_bom yes)
-		(on_board yes)
-		(dnp no)
-		(fields_autoplaced yes)
-		(property "Reference" "#PWR025"
-			(at 303.53 29.21 0)
-			(effects
-				(font
-					(size 1.27 1.27)
-				)
-				(hide yes)
-			)
-		)
-		(property "Value" "+5V"
-			(at 303.53 20.32 0)
-			(effects
-				(font
-					(size 1.27 1.27)
-				)
-			)
-		)
-		(property "Footprint" ""
-			(at 303.53 25.4 0)
-			(effects
-				(font
-					(size 1.27 1.27)
-				)
-				(hide yes)
-			)
-		)
-		(property "Datasheet" ""
-			(at 303.53 25.4 0)
-			(effects
-				(font
-					(size 1.27 1.27)
-				)
-				(hide yes)
-			)
-		)
-		(property "Description" "Power symbol creates a global label with name \"+5V\""
-			(at 303.53 25.4 0)
-			(effects
-				(font
-					(size 1.27 1.27)
-				)
-				(hide yes)
-			)
-		)
-		(pin "1"
-		)
-		(instances
-			(project "robocup2027-pcb-data"
-				(path "/fda8bdee-4e79-4e78-9174-7c0702f316a4"
-					(reference "#PWR025")
-					(unit 1)
-				)
-			)
-		)
-	)
-	(symbol
 		(lib_id "Motor:Motor_Servo")
 		(at 134.62 50.8 0)
@@
 			)
 		)
-		(property "Footprint" "ESP32-DEVKITC-32E:MODULE_ESP32-DEVKITC-32E"
+		(property "Footprint" "robo:MODULE_ESP32-DEVKITC-32E"
 			(at 114.3 146.05 0)
 			(effects
@@
 			)
 		)
-		(property "Footprint" "4-1437565-0:SW_4-1437565-0"
+		(property "Footprint" "robo:CW-SB11KKFF"
 			(at 86.36 133.35 0)
 			(effects
@@
 			)
 		)
-		(property "Footprint" "4-1437565-0:SW_4-1437565-0"
+		(property "Footprint" "robo:CW-SB11KKFF"
 			(at 38.1 38.1 0)
 			(effects
@@
 		)
 		(instances
-			(project ""
+			(project "robocup2027-pcb-data"
 				(path "/fda8bdee-4e79-4e78-9174-7c0702f316a4"
 					(reference "U17")
@@
 					(unit 1)
 				)
+			)
+		)
+	)
+	(symbol
+		(lib_id "power:+3.3V")
+		(at 303.53 25.4 0)
+		(unit 1)
+		(exclude_from_sim no)
+		(in_bom yes)
+		(on_board yes)
+		(dnp no)
+		(fields_autoplaced yes)
+		(property "Reference" "#PWR025"
+			(at 303.53 29.21 0)
+			(effects
+				(font
+					(size 1.27 1.27)
+				)
+				(hide yes)
+			)
+		)
+		(property "Value" "+3.3V"
+			(at 303.53 20.32 0)
+			(effects
+				(font
+					(size 1.27 1.27)
+				)
+			)
+		)
+		(property "Footprint" ""
+			(at 303.53 25.4 0)
+			(effects
+				(font
+					(size 1.27 1.27)
+				)
+				(hide yes)
+			)
+		)
+		(property "Datasheet" ""
+			(at 303.53 25.4 0)
+			(effects
+				(font
+					(size 1.27 1.27)
+				)
+				(hide yes)
+			)
+		)
+		(property "Description" "Power symbol creates a global label with name \"+3.3V\""
+			(at 303.53 25.4 0)
+			(effects
+				(font
+					(size 1.27 1.27)
+				)
+				(hide yes)
+			)
+		)
+		(pin "1"
+		)
+		(instances
+			(project "robocup2027-pcb-data"
+				(path "/fda8bdee-4e79-4e78-9174-7c0702f316a4"
+					(reference "#PWR025")
+					(unit 1)
+				)

Commit message: end of the day
Connections:
- net +3.3V: now also M5.2 (+), M6.2 (+)
- net +5V: no longer M5.2 (+), M6.2 (+)
Changed lines of the file:
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@@
+	)
+	(symbol
+		(lib_id "power:+3.3V")
+		(at 124.46 40.64 0)
+		(unit 1)
+		(exclude_from_sim no)
+		(in_bom yes)
+		(on_board yes)
+		(dnp no)
+		(fields_autoplaced yes)
+		(property "Reference" "#PWR017"
+			(at 124.46 44.45 0)
+			(effects
+				(font
+					(size 1.27 1.27)
+				)
+				(hide yes)
+			)
+		)
+		(property "Value" "+3.3V"
+			(at 124.46 35.56 0)
+			(effects
+				(font
+					(size 1.27 1.27)
+				)
+			)
+		)
+		(property "Footprint" ""
+			(at 124.46 40.64 0)
+			(effects
+				(font
+					(size 1.27 1.27)
+				)
+				(hide yes)
+			)
+		)
+		(property "Datasheet" ""
+			(at 124.46 40.64 0)
+			(effects
+				(font
+					(size 1.27 1.27)
+				)
+				(hide yes)
+			)
+		)
+		(property "Description" "Power symbol creates a global label with name \"+3.3V\""
+			(at 124.46 40.64 0)
+			(effects
+				(font
+					(size 1.27 1.27)
+				)
+				(hide yes)
+			)
+		)
+		(pin "1"
+		)
+		(instances
+			(project "robocup2027-pcb-data"
+				(path "/fda8bdee-4e79-4e78-9174-7c0702f316a4"
+					(reference "#PWR017")
+					(unit 1)
+				)
+			)
+		)
 	)
 	(symbol
@@
 					(unit 1)
 				)
-			)
-		)
-	)
-	(symbol
-		(lib_id "power:+5V")
-		(at 124.46 40.64 0)
-		(unit 1)
-		(exclude_from_sim no)
-		(in_bom yes)
-		(on_board yes)
-		(dnp no)
-		(fields_autoplaced yes)
-		(property "Reference" "#PWR017"
-			(at 124.46 44.45 0)
-			(effects
-				(font
-					(size 1.27 1.27)
-				)
-				(hide yes)
-			)
-		)
-		(property "Value" "+5V"
-			(at 124.46 35.56 0)
-			(effects
-				(font
-					(size 1.27 1.27)
-				)
-			)
-		)
-		(property "Footprint" ""
-			(at 124.46 40.64 0)
-			(effects
-				(font
-					(size 1.27 1.27)
-				)
-				(hide yes)
-			)
-		)
-		(property "Datasheet" ""
-			(at 124.46 40.64 0)
-			(effects
-				(font
-					(size 1.27 1.27)
-				)
-				(hide yes)
-			)
-		)
-		(property "Description" "Power symbol creates a global label with name \"+5V\""
-			(at 124.46 40.64 0)
-			(effects
-				(font
-					(size 1.27 1.27)
-				)
-				(hide yes)
-			)
-		)
-		(pin "1"
-		)
-		(instances
-			(project "robocup2027-pcb-data"
-				(path "/fda8bdee-4e79-4e78-9174-7c0702f316a4"
-					(reference "#PWR017")
-					(unit 1)
-				)

Commit message: fix pim
Connections:
- net FE-URT-2-RXD: now also U1.J3_11 (IO17); no longer U1.J3_12 (IO16)
- net FE-URT-2-TXD: now also U1.J3_12 (IO16); no longer U1.J3_11 (IO17)
